Commit message: update urdf and remove 2kg for lidar

File: b2_description/urdf/b2.urdf (robot description, URDF)
Before this commit: robot b2_description, 37 links, 36 joints
Links:
- link FR_hip: mass 2.256 -> 2.673
- link RL_hip: mass 2.256 -> 2.673
- link base_link: mass 35.86 -> 33.86; geometry collision box size=0.5 0.28 0.15; visual mesh filename=../meshes/base_link_no_lidar.dae
