Commit message: add general external force for b2 and b2g

File: robots/b2_description/urdf/b2.urdf (robot description, URDF)
Before this commit: robot b2_description, 37 links, 36 joints
Links:
- added link payload
Joints:
- added joint base_payload: type fixed, parent base_link, child payload, origin xyz=-0.25 0 0.075 rpy=0 0 0

Commit message: split b2 payload into front and rear, change arm z-velocity to global

File: robots/b2_description/urdf/b2.urdf (robot description, URDF)
Before this commit: robot b2_description, 38 links, 37 joints
Links:
- removed link payload
- added link payload_link_front
- added link payload_link_rear
Joints:
- removed joint base_payload
- added joint payload_joint_front: type fixed, parent base_link, child payload_link_front, origin xyz=0.19 0 0.20 rpy=0 0 0
- added joint payload_joint_rear: type fixed, parent base_link, child payload_link_rear, origin xyz=-0.25 0 0.075 rpy=0 0 0
